Commit message: Update KMU_robot.xacro
Исправлена ошибка при  использовании robot-state-publisher

File: KMU_robot_description/urdf/KMU_robot.xacro (robot description, xacro)
@@ -1,3 +1,3 @@
-<?xml version="1.0" ?>
+?xml version="1.0" ?>
 <robot name="KMU_robot" xmlns:xacro="http://www.ros.org/wiki/xacro">
 <xacro:include filename="$(find KMU_robot_description)/urdf/materials.xacro" />
@@ -13,5 +13,5 @@
     <origin xyz="0 0 0" rpy="0 0 0"/>
     <geometry>
-      <mesh filename="file://$(find KMU_robot_description)/meshes/base_link.stl" scale="0.001 0.001 0.001"/>
+      <mesh filename="package://KMU_robot_description/meshes/base_link.stl" scale="0.001 0.001 0.001"/>
     </geometry>
     <material name="silver"/>
@@ -20,5 +20,5 @@
     <origin xyz="0 0 0" rpy="0 0 0"/>
     <geometry>
-      <mesh filename="file://$(find KMU_robot_description)/meshes/base_link.stl" scale="0.001 0.001 0.001"/>
+      <mesh filename="package://KMU_robot_description/meshes/base_link.stl" scale="0.001 0.001 0.001"/>
     </geometry>
   </collision>
@@ -33,5 +33,5 @@
     <origin xyz="-0.0 0.151 -0.05" rpy="0 0 0"/>
     <geometry>
-      <mesh filename="file://$(find KMU_robot_description)/meshes/right_vel_1.stl" scale="0.001 0.001 0.001"/>
+      <mesh filename="package://KMU_robot_description/meshes/right_vel_1.stl" scale="0.001 0.001 0.001"/>
     </geometry>
     <material name="silver"/>
@@ -40,5 +40,5 @@
     <origin xyz="-0.0 0.151 -0.05" rpy="0 0 0"/>
     <geometry>
-      <mesh filename="file://$(find KMU_robot_description)/meshes/right_vel_1.stl" scale="0.001 0.001 0.001"/>
+      <mesh filename="package://KMU_robot_description/meshes/right_vel_1.stl" scale="0.001 0.001 0.001"/>
     </geometry>
   </collision>
@@ -53,5 +53,5 @@
     <origin xyz="-0.0 -0.151 -0.05" rpy="0 0 0"/>
     <geometry>
-      <mesh filename="file://$(find KMU_robot_description)/meshes/left_vel_1.stl" scale="0.001 0.001 0.001"/>
+      <mesh filename="package://KMU_robot_description/meshes/left_vel_1.stl" scale="0.001 0.001 0.001"/>
     </geometry>
     <material name="silver"/>
@@ -60,5 +60,5 @@
     <origin xyz="-0.0 -0.151 -0.05" rpy="0 0 0"/>
     <geometry>
-      <mesh filename="file://$(find KMU_robot_description)/meshes/left_vel_1.stl" scale="0.001 0.001 0.001"/>
+      <mesh filename="package://KMU_robot_description/meshes/left_vel_1.stl" scale="0.001 0.001 0.001"/>
     </geometry>
   </collision>
@@ -73,5 +73,5 @@
     <origin xyz="-0.0 -0.0 -0.16" rpy="0 0 0"/>
     <geometry>
-      <mesh filename="file://$(find KMU_robot_description)/meshes/lidar_1.stl" scale="0.001 0.001 0.001"/>
+      <mesh filename="package://KMU_robot_description/meshes/lidar_1.stl" scale="0.001 0.001 0.001"/>
     </geometry>
     <material name="silver"/>
@@ -80,5 +80,5 @@
     <origin xyz="-0.0 -0.0 -0.16" rpy="0 0 0"/>
     <geometry>
-      <mesh filename="file://$(find KMU_robot_description)/meshes/lidar_1.stl" scale="0.001 0.001 0.001"/>
+      <mesh filename="package://KMU_robot_description/meshes/lidar_1.stl" scale="0.001 0.001 0.001"/>
     </geometry>
   </collision>
